Commit message: update 14.01.25

File: robot_description/repair_full.urdf (robot description, URDF)
Before this commit: robot repair_full, 115 links, 114 joints
Joints:
- removed joint j_sliding_guide
- added joint j_torso_base: type prismatic, parent sliding_guide_link, child dummy_prismatic_link, origin xyz=0 0 0 rpy=0 0 0, axis 0 0 -1, limit lower=-1.0 upper=1.0 effort=147 velocity=5
- joint j_arm_1_7: origin xyz=0.0 -0.062877 0.05 rpy=1.570796326795 0.3316123 0.0 -> xyz=0.0 -0.062877 0.05 rpy=1.570796326795 0.0 0.0
- joint j_arm_2_7: origin xyz=0.0 0.062877 0.05 rpy=-1.570796326795 0.3316123 0.0 -> xyz=0.0 0.062877 0.05 rpy=-1.570796326795 0.0 0.0

Commit message: update 15.05.2025

File: robot_description/repair_full.urdf (robot description, URDF)
Before this commit: robot repair_full, 115 links, 114 joints
Links:
- link dummy_prismatic_link: mass None -> 0.0; geometry visual box size=0.1 0.1 1.0
Joints:
- joint j_torso_base: axis 0 0 -1 -> 0 0 1; limit lower=-1.0 upper=1.0 effort=147 velocity=5 -> lower=-1.0 upper=1.0 effort=147 velocity=2

Commit message: update 15.01.25

File: robot_description/repair_full.urdf (robot description, URDF)
Before this commit: robot repair_full, 115 links, 114 joints
Joints:
- joint j_torso_base: axis 0 0 -1 -> 0 0 1

Commit message: changes integration week september

File: robot_description/repair_full.urdf (robot description, URDF)
Before this commit: robot repair_full, 128 links, 127 joints
Joints:
- joint j_torso_base: origin xyz=0.0 0.0 0.0 rpy=0.0 0.0 0.0 -> xyz=0 0 0.07 rpy=0 0 0

Commit message: added danger zone

File: robot_description/repair_full.urdf (robot description, URDF)
Before this commit: robot repair_full, 128 links, 127 joints
Joints:
- joint j_torso_base: limit lower=-0.8 upper=0.8 effort=147.0 velocity=0.25 -> lower=-0.8 upper=0.8 effort=147.0 velocity=0.2

Commit message: old  but gold

File: robot_description/repair_full.urdf (robot description, URDF)
Before this commit: robot repair_full, 128 links, 127 joints
Links:
- removed link leg1_link
- removed link leg2_link
- removed link leg3_link
- removed link leg4_link
- removed link obar1_link
- removed link obar2_link
- removed link obar3_link
- removed link obar4_link
- removed link table_top_link
- removed link vbar1_link
- removed link vbar2_link
- removed link vbar3_link
- removed link vbar4_link
- link dummy_prismatic_link: mass 0.1 -> 0.0; geometry visual box size=0.1 0.1 1.0
Joints:
- removed joint leg1_joint
- removed joint leg2_joint
- removed joint leg3_joint
- removed joint leg4_joint
- removed joint obar1_joint
- removed joint obar2_joint
- removed joint obar3_joint
- removed joint obar4_joint
- removed joint table_top_link_joint
- removed joint vbar1_joint
- removed joint vbar2_joint
- removed joint vbar3_joint
- removed joint vbar4_joint
- joint j_torso_base: limit lower=-0.8 upper=0.8 effort=147.0 velocity=0.2 -> lower=-0.8 upper=0.8 effort=147 velocity=0.2
- joint sliding_guide_joint: origin xyz=0.0 1.25 0.3 rpy=-1.57079632679 0 0 -> xyz=-0.300 0.000 1.970 rpy=-1.571 -1.571 0.000; parent obar2_link -> world

Commit message: added translational limits, changed grasp link, and added active degree of freedom switch

File: robot_description/repair_full.urdf (robot description, URDF)
Before this commit: robot repair_full, 115 links, 114 joints
Links:
- added link leg1_link; collision cylinder length=0.978 radius=0.02; visual cylinder length=0.978 radius=0.02
- added link leg2_link; collision cylinder length=0.978 radius=0.02; visual cylinder length=0.978 radius=0.02
- added link leg3_link; collision cylinder length=0.978 radius=0.02; visual cylinder length=0.978 radius=0.02
- added link leg4_link; collision cylinder length=0.978 radius=0.02; visual cylinder length=0.978 radius=0.02
- added link obar1_link; collision cylinder length=1.0 radius=0.02; visual cylinder length=1.0 radius=0.02
- added link obar2_link; collision cylinder length=1.0 radius=0.02; visual cylinder length=1.0 radius=0.02
- added link obar3_link; collision cylinder length=2.5 radius=0.02; visual cylinder length=2.5 radius=0.02
- added link obar4_link; collision cylinder length=2.5 radius=0.02; visual cylinder length=2.5 radius=0.02
- added link table_top_link; collision box size=1.0 2.5 0.028; visual box size=1.0 2.5 0.028
- added link vbar1_link; collision cylinder length=0.97 radius=0.02; visual cylinder length=0.97 radius=0.02
- added link vbar2_link; collision cylinder length=0.97 radius=0.02; visual cylinder length=0.97 radius=0.02
- added link vbar3_link; collision cylinder length=0.97 radius=0.02; visual cylinder length=0.97 radius=0.02
- added link vbar4_link; collision cylinder length=0.97 radius=0.02; visual cylinder length=0.97 radius=0.02
- link dummy_prismatic_link: mass 0.0 -> 0.1; geometry 
Joints:
- added joint leg1_joint: type fixed, parent table_top_link, child leg1_link, origin xyz=0.5 1.25 0.978 rpy=0 0 0
- added joint leg2_joint: type fixed, parent table_top_link, child leg2_link, origin xyz=-0.5 1.25 0.978 rpy=0 0 0
- added joint leg3_joint: type fixed, parent table_top_link, child leg3_link, origin xyz=0.5 -1.25 0.978 rpy=0 0 0
- added joint leg4_joint: type fixed, parent table_top_link, child leg4_link, origin xyz=-0.5 -1.25 0.978 rpy=0 0 0
- added joint obar1_joint: type fixed, parent vbar1_link, child obar1_link, origin xyz=-0.5 0 0.485 rpy=0 -1.57079632679 0
- added joint obar2_joint: type fixed, parent vbar3_link, child obar2_link, origin xyz=-0.5 0 0.485 rpy=0 -1.57079632679 0
- added joint obar3_joint: type fixed, parent vbar3_link, child obar3_link, origin xyz=0 1.25 0.485 rpy=-1.57079632679 0 0
- added joint obar4_joint: type fixed, parent vbar4_link, child obar4_link, origin xyz=0 1.25 0.485 rpy=-1.57079632679 0 0
- added joint table_top_link_joint: type fixed, parent world, child table_top_link
- added joint vbar1_joint: type fixed, parent leg1_link, child vbar1_link, origin xyz=0 0 0.485 rpy=0 0 0
- added joint vbar2_joint: type fixed, parent leg2_link, child vbar2_link, origin xyz=0 0 0.485 rpy=0 0 0
- added joint vbar3_joint: type fixed, parent leg3_link, child vbar3_link, origin xyz=0 0 0.485 rpy=0 0 0
- added joint vbar4_joint: type fixed, parent leg4_link, child vbar4_link, origin xyz=0 0 0.485 rpy=0 0 0
- joint j_torso_base: limit lower=-0.8 upper=0.8 effort=147 velocity=0.2 -> lower=-0.7 upper=0.7 effort=147.0 velocity=0.2
- joint right_hand_v1_2_research_grasp_joint: origin xyz=-0.06 0.03 0.16 rpy=0 0 1.57 -> xyz=0.0 0.03 0.12 rpy=0 0 1.57
- joint sliding_guide_joint: origin xyz=-0.300 0.000 1.970 rpy=-1.571 -1.571 0.000 -> xyz=0.0 1.25 0.3 rpy=-1.57079632679 0 0; parent world -> obar2_link

Commit message: working state with fixed ramping  up and start config setting

File: robot_description/repair_full.urdf (robot description, URDF)
Before this commit: robot repair_full, 128 links, 127 joints
Joints:
- joint j_torso_base: limit lower=-0.7 upper=0.7 effort=147.0 velocity=0.2 -> lower=-0.75 upper=0.75 effort=147.0 velocity=0.05
- joint left_hand_v1_wide_grasp_joint: origin xyz=0.03 -0.10 0.15 rpy=0 0 0 -> xyz=0.05 -0.06 0.12 rpy=0 0 0
